Commit message: Created first model of Alfred

File: catkin_ws/src/sim/urdf/alfred.urdf (robot description, URDF)
Before this commit: robot Alfred, 1 links, 0 joints
Links:
- added link left_wheel; visual cylinder length=0.03 radius=0.035
- added link right_wheel; visual cylinder length=0.03 radius=0.035
- link base_link: geometry visual box size=0.15 0.07 0.10
Joints:
- added joint base_to_left_wheel: type fixed, parent base_link, child left_wheel, origin xyz=0 0 0.035
- added joint base_to_right_wheel: type fixed, parent base_link, child right_wheel, origin xyz=0 0 0.035

Commit message: Created first model of Alfred

File: catkin_ws/src/sim/urdf/alfred.urdf (robot description, URDF)
Before this commit: robot Alfred, 3 links, 2 joints
Joints:
- joint base_to_left_wheel: axis (none) -> 0 1 0; limit (none) -> lower=0.0 upper=0.548 effort=1000.0 velocity=0.5; type fixed -> revolute
- joint base_to_right_wheel: axis (none) -> 0 1 0; limit (none) -> lower=0.0 upper=0.548 effort=1000.0 velocity=0.5; type fixed -> revolute

Commit message: Corrected axis for wheel joints

File: catkin_ws/src/sim/urdf/alfred.urdf (robot description, URDF)
Before this commit: robot Alfred, 3 links, 2 joints
Joints:
- joint base_to_left_wheel: axis 0 1 0 -> 1 0 0; limit lower=0.0 upper=0.548 effort=1000.0 velocity=0.5 -> (none)
- joint base_to_right_wheel: axis 0 1 0 -> 1 0 0; limit lower=0.0 upper=0.548 effort=1000.0 velocity=0.5 -> (none)

Commit message: Added collision element in URDF

File: catkin_ws/src/sim/urdf/alfred.urdf (robot description, URDF)
Before this commit: robot Alfred, 3 links, 2 joints
Links:
- link base_link: geometry collision box size=0.15 0.07 0.10; visual box size=0.15 0.07 0.10
- link left_wheel: geometry collision cylinder length=0.03 radius=0.035; visual cylinder length=0.03 radius=0.035
- link right_wheel: geometry collision cylinder length=0.03 radius=0.035; visual cylinder length=0.03 radius=0.035

Commit message: Added inertial element in URDF

File: catkin_ws/src/sim/urdf/alfred.urdf (robot description, URDF)
Before this commit: robot Alfred, 3 links, 2 joints
Links:
- link base_link: mass None -> 1
- link left_wheel: mass None -> 0.03
- link right_wheel: mass None -> 0.03

Commit message: Created simulation under Gazebo

File: catkin_ws/src/sim/urdf/alfred.urdf (robot description, URDF)
Before this commit: robot Alfred, 3 links, 2 joints
Links:
- added link dummy
Joints:
- added joint dummy_joint: type fixed, parent dummy, child base_link
- joint base_to_left_wheel: origin xyz=0 0 0.035 -> xyz=-0.09 0 -0.035; type revolute -> continuous
- joint base_to_right_wheel: origin xyz=0 0 0.035 -> xyz=0.09 0 -0.035; type revolute -> continuous
