Commit message: Now using xacro instead of classical urdf description

File: catkin_ws/src/sim/urdf/alfred.xacro (robot description, xacro)
@@ -1,4 +1,4 @@
 <?xml version="1.0"?>
-<robot name="Alfred">
+<robot name="Alfred" xmlns:xacro="http://www.ros.org/wiki/xacro">
   <material name="blue">
     <color rgba="0 0 0.8 1"/>
@@ -7,4 +7,10 @@
     <color rgba="0 0 0 1"/>
   </material>
+  <xacro:property name="bodyLength" value="0.15" />
+  <xacro:property name="bodyHeight" value="0.10" />
+  <xacro:property name="bodyDepth" value="0.07" />
+  <xacro:property name="wheelRadius" value="0.035" />
+  <xacro:property name="wheelWidth" value="0.03" />
+  <xacro:property name="pi_2" value="1.57075" />
   <link name="dummy">
   </link>
@@ -12,13 +18,11 @@
     <visual>
       <geometry>
-        <box size="0.15 0.07 0.10" />
+        <box size="${bodyLength} ${bodyDepth} ${bodyHeight}" />
       </geometry>
-      <origin rpy="0 0 0" xyz="0 0 0"/>
       <material name="black"/>
     </visual>
     <collision>
       <geometry>
-        <box size="0.15 0.07 0.10" />
-        <origin rpy="0 0 0" xyz="0 0 0"/>
+        <box size="${bodyLength} ${bodyDepth} ${bodyHeight}" />
       </geometry>
     </collision>
@@ -32,56 +36,36 @@
     <child link="base_link"/>
   </joint>
-  <link name="right_wheel">
-    <visual>
-      <geometry>
-        <cylinder length="0.03" radius="0.035"/>
-      </geometry>
-      <origin rpy="0 1.57075 0" xyz="0 0 0"/>
-      <material name="blue"/>
-    </visual>
-    <collision>
-      <geometry>
-        <cylinder length="0.03" radius="0.035"/>
-      </geometry>
-      <origin rpy="0 1.57075 0" xyz="0 0 0"/>
-    </collision>
-    <inertial>
-      <mass value="0.03"/>
-      <inertia ixx="1.14e-5" ixy="0.0" ixz="0.0" iyy="1.14e-5" iyz="0.0" izz="1.84e-5"/>
-    </inertial>
-  </link>
-  <gazebo reference="right_wheel">
-    <mu1 value="200.0"/>
-    <mu2 value="100.0"/>
-    <kp value="10000000.0" />
-    <kd value="1.0" />
-    <material>Gazebo/Grey</material>
-  </gazebo>
-  <link name="left_wheel">
-    <visual>
-      <geometry>
-        <cylinder length="0.03" radius="0.035"/>
-      </geometry>
-      <origin rpy="0 1.57075 0" xyz="0 0 0"/>
-      <material name="blue"/>
-    </visual>
-    <collision>
-      <geometry>
-        <cylinder length="0.03" radius="0.035"/>
-      </geometry>
-      <origin rpy="0 1.57075 0" xyz="0 0 0"/>
-    </collision>
-    <inertial>
-      <mass value="0.03"/>
-      <inertia ixx="1.14e-5" ixy="0.0" ixz="0.0" iyy="1.14e-5" iyz="0.0" izz="1.84e-5"/>
-    </inertial>
-  </link>
-  <gazebo reference="left_wheel">
-    <mu1 value="200.0"/>
-    <mu2 value="100.0"/>
-    <kp value="10000000.0" />
-    <kd value="1.0" />
-    <material>Gazebo/Grey</material>
-  </gazebo>
+  <xacro:macro name="wheel" params="side">
+    <link name="${side}_wheel">
+      <visual>
+        <geometry>
+          <cylinder length="${wheelWidth}" radius="${wheelRadius}"/>
+        </geometry>
+        <origin rpy="0 ${pi_2} 0" xyz="0 0 0"/>
+        <material name="blue"/>
+      </visual>
+      <collision>
+        <geometry>
+          <cylinder length="${wheelWidth}" radius="${wheelRadius}"/>
+        </geometry>
+        <origin rpy="0 ${pi_2} 0" xyz="0 0 0"/>
+      </collision>
+      <inertial>
+        <mass value="0.03"/>
+        <inertia ixx="1.14e-5" ixy="0.0" ixz="0.0" iyy="1.14e-5" iyz="0.0" izz="1.84e-5"/>
+      </inertial>
+    </link>
+    <gazebo reference="${side}_wheel">
+      <mu1 value="200.0"/>
+      <mu2 value="100.0"/>
+      <kp value="10000000.0" />
+      <kd value="1.0" />
+      <material>Gazebo/Grey</material>
+    </gazebo>
+  </xacro:macro>
+  <xacro:wheel side="right">
+  </xacro:wheel>
+  <xacro:wheel side="left">
+  </xacro:wheel>
   <joint name="base_to_right_wheel" type="continuous">
     <parent link="base_link"/>

Commit message: Made xacro macros prettier

File: catkin_ws/src/sim/urdf/alfred.xacro (robot description, xacro)
@@ -7,51 +7,47 @@
     <color rgba="0 0 0 1"/>
   </material>
+<!-- Physical definition -->
   <xacro:property name="bodyLength" value="0.15" />
   <xacro:property name="bodyHeight" value="0.10" />
   <xacro:property name="bodyDepth" value="0.07" />
+  <xacro:property name="bodyMass" value="1" />
   <xacro:property name="wheelRadius" value="0.035" />
   <xacro:property name="wheelWidth" value="0.03" />
+  <xacro:property name="wheelMass" value="0.03" />
   <xacro:property name="pi_2" value="1.57075" />
-  <link name="dummy">
-  </link>
-  <link name="base_link">
-    <visual>
-      <geometry>
-        <box size="${bodyLength} ${bodyDepth} ${bodyHeight}" />
-      </geometry>
-      <material name="black"/>
-    </visual>
-    <collision>
-      <geometry>
-        <box size="${bodyLength} ${bodyDepth} ${bodyHeight}" />
-      </geometry>
-    </collision>
-    <inertial>
-      <mass value="1"/>
-      <inertia ixx="1.24e-3" ixy="0.0" ixz="0.0" iyy="2.28e-3" iyz="0.0" izz="2.71e-3"/>
-    </inertial>
-  </link>
-  <joint name="dummy_joint" type="fixed">
-    <parent link="dummy"/>
-    <child link="base_link"/>
-  </joint>
-  <xacro:macro name="wheel" params="side">
+<!-- Macros definition -->
+  <xacro:macro name="body_shape">
+    <geometry>
+      <box size="${bodyLength} ${bodyDepth} ${bodyHeight}" />
+    </geometry>
+  </xacro:macro>
+  <xacro:macro name="wheel_shape">
+    <geometry>
+      <cylinder length="${wheelWidth}" radius="${wheelRadius}"/>
+    </geometry>
+    <origin rpy="0 ${pi_2} 0" xyz="0 0 0"/>
+  </xacro:macro>
+  <xacro:macro name="cylinder_inertia" params="radius height mass">
+    <mass value="${mass}"/>
+    <inertia ixx="${1/12*mass*(radius*radius+height*height)}" ixy="0.0" ixz="0.0" iyy="${1/12*mass*(radius*radius+height*height)}" iyz="0.0" izz="${1/12*mass*radius*radius}"/>
+  </xacro:macro>
+  <xacro:macro name="box_inertia" params="width height depth mass">
+    <mass value="${mass}"/>
+    <inertia ixx="${1/12*mass*(height*height+depth*depth)}" ixy="0.0" ixz="0.0" iyy="${1/12*mass*(width*width+depth*depth)}" iyz="0.0" izz="${1/12*mass*(width*width+height*height)}"/>
+  </xacro:macro>
+  <xacro:macro name="wheel_link" params="side">
     <link name="${side}_wheel">
       <visual>
-        <geometry>
-          <cylinder length="${wheelWidth}" radius="${wheelRadius}"/>
-        </geometry>
-        <origin rpy="0 ${pi_2} 0" xyz="0 0 0"/>
+        <xacro:wheel_shape>
+        </xacro:wheel_shape>
         <material name="blue"/>
       </visual>
       <collision>
-        <geometry>
-          <cylinder length="${wheelWidth}" radius="${wheelRadius}"/>
-        </geometry>
-        <origin rpy="0 ${pi_2} 0" xyz="0 0 0"/>
+        <xacro:wheel_shape>
+        </xacro:wheel_shape>
       </collision>
       <inertial>
-        <mass value="0.03"/>
-        <inertia ixx="1.14e-5" ixy="0.0" ixz="0.0" iyy="1.14e-5" iyz="0.0" izz="1.84e-5"/>
+        <xacro:cylinder_inertia radius="${wheelRadius}" height="${wheelWidth}" mass="${wheelMass}">
+        </xacro:cylinder_inertia>
       </inertial>
     </link>
@@ -64,8 +60,42 @@
     </gazebo>
   </xacro:macro>
-  <xacro:wheel side="right">
-  </xacro:wheel>
-  <xacro:wheel side="left">
-  </xacro:wheel>
+  <xacro:macro name="wheel_transmission" params="side">
+    <transmission name="${side}_wheel_rotation">
+      <type>transmission_interface/SimpleTransmission</type>
+      <actuator name="${side}_wheel_motor">
+        <mechanicalReduction>1</mechanicalReduction>
+      </actuator>
+      <joint name="base_to_${side}_wheel">
+        <hardwareInterface>hardware_interface/VelocityJointInterface</hardwareInterface>
+      </joint>
+    </transmission>
+  </xacro:macro>
+<!-- Links definition -->
+  <link name="dummy">
+  </link>
+  <link name="base_link">
+    <visual>
+      <xacro:body_shape>
+      </xacro:body_shape>
+      <material name="black"/>
+    </visual>
+    <collision>
+      <xacro:body_shape>
+      </xacro:body_shape>
+    </collision>
+    <inertial>
+      <xacro:box_inertia width="${bodyLength}" height="${bodyHeight}" depth ="${bodyDepth}" mass="${bodyMass}">
+      </xacro:box_inertia>
+    </inertial>
+  </link>
+  <xacro:wheel_link side="right">
+  </xacro:wheel_link>
+  <xacro:wheel_link side="left">
+  </xacro:wheel_link>
+<!-- Joints definition -->
+  <joint name="dummy_joint" type="fixed">
+    <parent link="dummy"/>
+    <child link="base_link"/>
+  </joint>
   <joint name="base_to_right_wheel" type="continuous">
     <parent link="base_link"/>
@@ -74,13 +104,4 @@
     <axis xyz="1 0 0"/>
   </joint>
-  <transmission name="right_wheel_rotation">
-    <type>transmission_interface/SimpleTransmission</type>
-    <actuator name="$right_wheel_motor">
-      <mechanicalReduction>1</mechanicalReduction>
-    </actuator>
-    <joint name="base_to_right_wheel">
-      <hardwareInterface>hardware_interface/VelocityJointInterface</hardwareInterface>
-    </joint>
-  </transmission>
   <joint name="base_to_left_wheel" type="continuous">
     <parent link="base_link"/>
@@ -89,14 +110,10 @@
     <axis xyz="1 0 0"/>
   </joint>
-  <transmission name="left_wheel_rotation">
-    <type>transmission_interface/SimpleTransmission</type>
-    <actuator name="$left_wheel_motor">
-      <mechanicalReduction>1</mechanicalReduction>
-    </actuator>
-    <joint name="base_to_left_wheel">
-      <hardwareInterface>hardware_interface/VelocityJointInterface</hardwareInterface>
-    </joint>
-  </transmission>
-  <!-- Gazebo plugin for ROS Control -->
+<!-- Wheels transmission definition -->
+  <xacro:wheel_transmission side="right">
+  </xacro:wheel_transmission>
+  <xacro:wheel_transmission side="left">
+  </xacro:wheel_transmission>
+<!-- Gazebo plugin for ROS Control -->
   <gazebo>
     <plugin name="gazebo_ros_control" filename="libgazebo_ros_control.so">

Commit message: Used pi value instead of hard coded value

File: catkin_ws/src/sim/urdf/alfred.xacro (robot description, xacro)
@@ -7,5 +7,5 @@
     <color rgba="0 0 0 1"/>
   </material>
-<!-- Physical definition -->
+<!-- Physical definitions -->
   <xacro:property name="bodyLength" value="0.15" />
   <xacro:property name="bodyHeight" value="0.10" />
@@ -15,5 +15,4 @@
   <xacro:property name="wheelWidth" value="0.03" />
   <xacro:property name="wheelMass" value="0.03" />
-  <xacro:property name="pi_2" value="1.57075" />
 <!-- Macros definition -->
   <xacro:macro name="body_shape">
@@ -26,5 +25,5 @@
       <cylinder length="${wheelWidth}" radius="${wheelRadius}"/>
     </geometry>
-    <origin rpy="0 ${pi_2} 0" xyz="0 0 0"/>
+    <origin rpy="0 ${pi/2} 0" xyz="0 0 0"/>
   </xacro:macro>
   <xacro:macro name="cylinder_inertia" params="radius height mass">

Commit message: Cleaned urdf file

File: catkin_ws/src/sim/urdf/alfred.xacro (robot description, xacro)
@@ -15,4 +15,6 @@
   <xacro:property name="wheelWidth" value="0.03" />
   <xacro:property name="wheelMass" value="0.03" />
+  <xacro:property name="rightWheelXPos" value="-0.09" />
+  <xacro:property name="leftWheelXPos" value="0.09" />
 <!-- Macros definition -->
   <xacro:macro name="body_shape">
@@ -29,5 +31,5 @@
   <xacro:macro name="cylinder_inertia" params="radius height mass">
     <mass value="${mass}"/>
-    <inertia ixx="${1/12*mass*(radius*radius+height*height)}" ixy="0.0" ixz="0.0" iyy="${1/12*mass*(radius*radius+height*height)}" iyz="0.0" izz="${1/12*mass*radius*radius}"/>
+    <inertia ixx="${1/12*mass*(3*radius*radius+height*height)}" ixy="0.0" ixz="0.0" iyy="${1/12*mass*(3*radius*radius+height*height)}" iyz="0.0" izz="${1/2*mass*radius*radius}"/>
   </xacro:macro>
   <xacro:macro name="box_inertia" params="width height depth mass">
@@ -38,15 +40,12 @@
     <link name="${side}_wheel">
       <visual>
-        <xacro:wheel_shape>
-        </xacro:wheel_shape>
+        <xacro:wheel_shape />
         <material name="blue"/>
       </visual>
       <collision>
-        <xacro:wheel_shape>
-        </xacro:wheel_shape>
+        <xacro:wheel_shape />
       </collision>
       <inertial>
-        <xacro:cylinder_inertia radius="${wheelRadius}" height="${wheelWidth}" mass="${wheelMass}">
-        </xacro:cylinder_inertia>
+        <xacro:cylinder_inertia radius="${wheelRadius}" height="${wheelWidth}" mass="${wheelMass}" />
       </inertial>
     </link>
@@ -70,4 +69,17 @@
     </transmission>
   </xacro:macro>
+  <xacro:macro name="wheel_joint" params="side">
+    <joint name="base_to_${side}_wheel" type="continuous">
+      <parent link="base_link"/>
+      <child link="${side}_wheel"/>
+      <xacro:if value="${side == 'right'}" >
+        <origin xyz="${rightWheelXPos} 0 ${-wheelRadius}"/>
+      </xacro:if>
+      <xacro:if value="${side == 'left'}" >
+        <origin xyz="${leftWheelXPos} 0 ${-wheelRadius}"/>
+      </xacro:if>
+      <axis xyz="1 0 0"/>
+    </joint>
+  </xacro:macro>
 <!-- Links definition -->
   <link name="dummy">
@@ -75,21 +87,16 @@
   <link name="base_link">
     <visual>
-      <xacro:body_shape>
-      </xacro:body_shape>
+      <xacro:body_shape />
       <material name="black"/>
     </visual>
     <collision>
-      <xacro:body_shape>
-      </xacro:body_shape>
+      <xacro:body_shape />
     </collision>
     <inertial>
-      <xacro:box_inertia width="${bodyLength}" height="${bodyHeight}" depth ="${bodyDepth}" mass="${bodyMass}">
-      </xacro:box_inertia>
+      <xacro:box_inertia width="${bodyLength}" height="${bodyHeight}" depth ="${bodyDepth}" mass="${bodyMass}" />
     </inertial>
   </link>
-  <xacro:wheel_link side="right">
-  </xacro:wheel_link>
-  <xacro:wheel_link side="left">
-  </xacro:wheel_link>
+  <xacro:wheel_link side="right" />
+  <xacro:wheel_link side="left" />
 <!-- Joints definition -->
   <joint name="dummy_joint" type="fixed">
@@ -97,21 +104,9 @@
     <child link="base_link"/>
   </joint>
-  <joint name="base_to_right_wheel" type="continuous">
-    <parent link="base_link"/>
-    <child link="right_wheel"/>
-    <origin xyz="0.09 0 -0.035"/>
-    <axis xyz="1 0 0"/>
-  </joint>
-  <joint name="base_to_left_wheel" type="continuous">
-    <parent link="base_link"/>
-    <child link="left_wheel"/>
-    <origin xyz="-0.09 0 -0.035"/>
-    <axis xyz="1 0 0"/>
-  </joint>
+  <xacro:wheel_joint side="right" />
+  <xacro:wheel_joint side="left" />
 <!-- Wheels transmission definition -->
-  <xacro:wheel_transmission side="right">
-  </xacro:wheel_transmission>
-  <xacro:wheel_transmission side="left">
-  </xacro:wheel_transmission>
+  <xacro:wheel_transmission side="right" />
+  <xacro:wheel_transmission side="left" />
 <!-- Gazebo plugin for ROS Control -->
   <gazebo>

Commit message: Updated physical measurements in urdf file

File: catkin_ws/src/sim/urdf/alfred.xacro (robot description, xacro)
@@ -11,12 +11,13 @@
 <!-- #################### -->
   <xacro:property name="bodyLength" value="0.15" />
-  <xacro:property name="bodyHeight" value="0.10" />
-  <xacro:property name="bodyDepth" value="0.07" />
-  <xacro:property name="bodyMass" value="1" />
-  <xacro:property name="wheelRadius" value="0.035" />
-  <xacro:property name="wheelWidth" value="0.03" />
-  <xacro:property name="wheelMass" value="0.03" />
-  <xacro:property name="rightWheelXPos" value="-0.09" />
-  <xacro:property name="leftWheelXPos" value="0.09" />
+  <xacro:property name="bodyHeight" value="0.11" />
+  <xacro:property name="bodyDepth" value="0.09" />
+  <xacro:property name="bodyMass" value="0.72" />
+  <xacro:property name="wheelRadius" value="0.0375" />
+  <xacro:property name="wheelWidth" value="0.035" />
+  <xacro:property name="wheelMass" value="0.05" />
+  <xacro:property name="rightWheelXPos" value="-0.09375" />
+  <xacro:property name="leftWheelXPos" value="0.09375" />
+  <xacro:property name="wheelZPos" value="-0.04" />
 <!-- ################# -->
 <!-- Macros definition -->
@@ -85,8 +86,8 @@
       <child link="${side}_wheel"/>
       <xacro:if value="${side == 'right'}" >
-        <origin xyz="${rightWheelXPos} 0 ${-wheelRadius}"/>
+        <origin xyz="${rightWheelXPos} 0 ${wheelZPos}"/>
       </xacro:if>
       <xacro:if value="${side == 'left'}" >
-        <origin xyz="${leftWheelXPos} 0 ${-wheelRadius}"/>
+        <origin xyz="${leftWheelXPos} 0 ${wheelZPos}"/>
       </xacro:if>
       <axis xyz="1 0 0"/>

Commit message: Updated masses of parts

File: catkin_ws/src/sim/urdf/alfred.xacro (robot description, xacro)
@@ -13,8 +13,8 @@
   <xacro:property name="bodyHeight" value="0.11" />
   <xacro:property name="bodyDepth" value="0.09" />
-  <xacro:property name="bodyMass" value="0.72" />
+  <xacro:property name="bodyMass" value="0.69" />
   <xacro:property name="wheelRadius" value="0.0375" />
   <xacro:property name="wheelWidth" value="0.035" />
-  <xacro:property name="wheelMass" value="0.05" />
+  <xacro:property name="wheelMass" value="0.065" />
   <xacro:property name="rightWheelXPos" value="-0.09375" />
   <xacro:property name="leftWheelXPos" value="0.09375" />
